File: sh-xi/hullo_road/control_board_template.kicad_pcb (KiCad board)
At the start: 2 copper layers, 230.5 x 80.6 mm, 541 parts, among them J1 Conn_01x16_Socket, J2 Conn_01x16_Socket, J3 Conn_01x16_Socket, J4 Conn_01x16_Pin, J5 Conn_01x16_Pin, J6 Conn_01x16_Pin, U1 ATtiny414-SS, U2 74HC595, U3 74HC595, U4 74HC595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

Commit message: Create two board design and route most things
Parts:
- added J4: Conn_01x16_Pin, Connector_PinHeader_2.54mm:PinHeader_1x16_P2.54mm_Vertical, F.Cu at (417.9, 40.2)
- added J5: Conn_01x16_Pin, Connector_PinHeader_2.54mm:PinHeader_1x16_P2.54mm_Vertical, F.Cu at (422.9, 32.6)
- added J6: Conn_01x16_Pin, Connector_PinHeader_2.54mm:PinHeader_1x16_P2.54mm_Vertical, F.Cu at (477.5, 32.6)
- moved U1 28.6 mm to (211.5, 84.5)
- moved U7 9.46 mm to (230.7, 64.4)
- moved U6 6.00 mm to (213.0, 62.5)
Routing:
- net +5V: track 157.3 -> 87.7 mm, vias 7 -> 4
- net CS_CP: track 87.1 -> 26.5 mm, vias 5 -> 2
- net CCol31: track 36.6 -> 0.00 mm
- net CCol30: track 34.8 -> 0.00 mm
- net CCol29: track 33.0 -> 0.00 mm
- net Net-(U5-QH'): track 34.0 -> 1.96 mm, vias 2 -> 1
- net CCol28: track 31.2 -> 0.00 mm
- net CCol23: track 30.0 -> 0.00 mm
- net CCol27: track 29.4 -> 0.00 mm
- net CCol22: track 28.2 -> 0.00 mm
- net CCol26: track 27.3 -> 0.00 mm
- net CCol21: track 26.4 -> 0.00 mm
- net CCol17: track 26.0 -> 0.00 mm
- net CCol18: track 25.8 -> 0.00 mm
- net CCol25: track 25.0 -> 0.00 mm
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Other:
- board size 230.5 x 80.6 mm -> 504.5 x 80.6 mm
